File: 20 - STM32_BOARD/stm32_board/GPP.sch (KiCad schematic (older format))
At the start: 2 parts, among them J1 Conn_01x04, J2 Conn_01x04

Commit message: stm32
Parts:
- added R? (x2): 100, symbol Device:R_Small
Connections:
- net LD1_RXi: now also R?.1; no longer J1.2 (Pin_2), J2.2 (Pin_2)
- net LD1_TXo: now also R?.1; no longer J1.3 (Pin_3), J2.3 (Pin_3)
- new net: J1.2 (Pin_2), J2.2 (Pin_2), R?.2
- new net: J1.3 (Pin_3), J2.3 (Pin_3), R?.2
Other:
- moved on the sheet: J1, J2
Changed lines of the file:
@@
 L Connector_Generic:Conn_01x04 J1
 U 1 1 5DA17A2F
-P 950 7200
-F 0 "J1" H 869 7514 50  0000 C CNN
-F 1 "Conn_01x04" H 869 7425 50  0000 C CNN
-F 2 "Connectors_JST:JST_SH_SM04B-SRSS-TB_04x1.00mm_Angled" H 950 7200 50  0001 C CNN
-F 3 "~" H 950 7200 50  0001 C CNN
-	1    950  7200
+P 800 6400
+F 0 "J1" H 719 6714 50  0000 C CNN
+F 1 "Conn_01x04" H 719 6625 50  0000 C CNN
+F 2 "Connectors_JST:JST_SH_SM04B-SRSS-TB_04x1.00mm_Angled" H 800 6400 50  0001 C CNN
+F 3 "~" H 800 6400 50  0001 C CNN
+	1    800  6400
 	-1   0    0    -1
 $EndComp
-Text Label 1150 7100 0    50   ~ 0
+Text Label 1000 6300 0    50   ~ 0
 5V_LIDAR
-Text Label 1150 7200 0    50   ~ 0
-LD1_RXi
-Text Label 1150 7300 0    50   ~ 0
-LD1_TXo
 $Comp
 L power:GND #PWR0101
 U 1 1 5DA196C0
-P 1200 7450
-F 0 "#PWR0101" H 1200 7200 50  0001 C CNN
-F 1 "GND" H 1205 7279 50  0000 C CNN
-F 2 "" H 1200 7450 50  0001 C CNN
-F 3 "" H 1200 7450 50  0001 C CNN
-	1    1200 7450
+P 1050 6650
+F 0 "#PWR0101" H 1050 6400 50  0001 C CNN
+F 1 "GND" H 1055 6479 50  0000 C CNN
+F 2 "" H 1050 6650 50  0001 C CNN
+F 3 "" H 1050 6650 50  0001 C CNN
+	1    1050 6650
 	1    0    0    -1
 $EndComp
 Wire Wire Line
-	1150 7400 1200 7400
+	1000 6600 1050 6600
 Wire Wire Line
-	1200 7400 1200 7450
+	1050 6600 1050 6650
 $Comp
 L Connector_Generic:Conn_01x04 J2
 U 1 1 5DA19F56
-P 1650 7200
-F 0 "J2" H 1569 7514 50  0000 C CNN
-F 1 "Conn_01x04" H 1569 7425 50  0000 C CNN
-F 2 "Pin_Headers:Pin_Header_Straight_1x04_Pitch2.54mm" H 1650 7200 50  0001 C CNN
-F 3 "~" H 1650 7200 50  0001 C CNN
-	1    1650 7200
+P 800 7150
+F 0 "J2" H 719 7464 50  0000 C CNN
+F 1 "Conn_01x04" H 719 7375 50  0000 C CNN
+F 2 "Pin_Headers:Pin_Header_Straight_1x04_Pitch2.54mm" H 800 7150 50  0001 C CNN
+F 3 "~" H 800 7150 50  0001 C CNN
+	1    800  7150
 	-1   0    0    -1
 $EndComp
-Text Label 1850 7100 0    50   ~ 0
+Text Label 1000 7050 0    50   ~ 0
 5V_LIDAR
-Text Label 1850 7200 0    50   ~ 0
+Text Label 2050 6400 0    50   ~ 0
 LD1_RXi
-Text Label 1850 7300 0    50   ~ 0
+Text Label 2050 6500 0    50   ~ 0
 LD1_TXo
 $Comp
 L power:GND #PWR0102
 U 1 1 5DA19F63
-P 1900 7450
-F 0 "#PWR0102" H 1900 7200 50  0001 C CNN
-F 1 "GND" H 1905 7279 50  0000 C CNN
-F 2 "" H 1900 7450 50  0001 C CNN
-F 3 "" H 1900 7450 50  0001 C CNN
-	1    1900 7450
+P 1050 7400
+F 0 "#PWR0102" H 1050 7150 50  0001 C CNN
+F 1 "GND" H 1055 7229 50  0000 C CNN
+F 2 "" H 1050 7400 50  0001 C CNN
+F 3 "" H 1050 7400 50  0001 C CNN
+	1    1050 7400
 	1    0    0    -1
 $EndComp
 Wire Wire Line
-	1850 7400 1900 7400
+	1000 7350 1050 7350
 Wire Wire Line
-	1900 7400 1900 7450
+	1050 7350 1050 7400
+$Comp
+L Device:R_Small R?
+U 1 1 5DA18202
+P 1800 6400
+F 0 "R?" V 1607 6400 50  0000 C CNN
+F 1 "100" V 1696 6400 50  0000 C CNN
+F 2 "" H 1800 6400 50  0001 C CNN
+F 3 "~" H 1800 6400 50  0001 C CNN
+	1    1800 6400
+	0    1    1    0
+$EndComp
+$Comp
+L Device:R_Small R?
+U 1 1 5DA19838
+P 1800 6500
+F 0 "R?" V 1607 6500 50  0000 C CNN
+F 1 "100" V 1696 6500 50  0000 C CNN
+F 2 "" H 1800 6500 50  0001 C CNN
+F 3 "~" H 1800 6500 50  0001 C CNN
+	1    1800 6500
+	0    1    1    0
+$EndComp
+Wire Wire Line
+	1000 6400 1450 6400
+Wire Wire Line
+	1000 6500 1550 6500
+Wire Wire Line
+	1450 7150 1450 6400
+Wire Wire Line
+	1000 7150 1450 7150
+Connection ~ 1450 6400
+Wire Wire Line
+	1450 6400 1700 6400
+Wire Wire Line
+	1550 7250 1550 6500
+Wire Wire Line
+	1000 7250 1550 7250
+Connection ~ 1550 6500
+Wire Wire Line
+	1550 6500 1700 6500
+Wire Wire Line
+	1900 6400 2050 6400
+Wire Wire Line
+	1900 6500 2050 6500
 $EndSCHEMATC

Commit message: stm32
Parts:
- added J? (x3): Conn_01x04, Connectors_JST:JST_SH_SM04B-SRSS-TB_04x1.00mm_Angled, symbol Connector_Generic:Conn_01x04
- added J? (x3): Conn_01x04, Pin_Headers:Pin_Header_Straight_1x04_Pitch2.54mm, symbol Connector_Generic:Conn_01x04
- added J?: Conn_01x03, symbol Connector_Generic:Conn_01x03
- added J?: Conn_01x09, symbol Connector_Generic:Conn_01x09
- added R? (x6): 100, symbol Device:R_Small
Connections:
- net 5V_LIDAR: now also J?.1 (Pin_1), J?.1 (Pin_1), J?.1 (Pin_1), J?.1 (Pin_1), J?.1 (Pin_1), J?.1 (Pin_1), J?.2 (Pin_2)
- net GND: now also J?.3 (Pin_3), J?.4 (Pin_4), J?.4 (Pin_4), J?.4 (Pin_4), J?.4 (Pin_4), J?.4 (Pin_4), J?.4 (Pin_4), J?.7 (Pin_7)
- net LD1_RXi: now also R?.1; no longer R?.1
- net LD1_TXo: now also R?.1; no longer R?.1
- new net: J?.2 (Pin_2), J?.2 (Pin_2), R?.2 (x3)
- new net: J?.3 (Pin_3), J?.3 (Pin_3), R?.2 (x3)
- new net 3V_LDO_GPS: J?.8 (Pin_8)
- new net GPS_ENo: J?.2 (Pin_2)
- new net GPS_FIXi: J?.4 (Pin_4)
- new net GPS_PPSi: J?.9 (Pin_9)
- new net GPS_RXi: J?.5 (Pin_5)
- new net GPS_TXo: J?.6 (Pin_6)
- new net LD2_RXi: R?.1
- new net LD2_TXo: R?.1
- new net LD3_RXi: R?.1
- new net LD3_TXo: R?.1
- new net LD4_RXi: R?.1
- new net LD4_TXo: R?.1
- new net VBATT: J?.3 (Pin_3)
- no-connect marks 0 -> 2
Other:
- note added: "LDO 3.3V pour GPS à partir du BEC"
- note added: "LIDAR"
- note added: "Partager les liaisons séries de telle sorte que les DMA sont disponible pour le RPLIDAR ou pour les 4 LIDAR"
- moved on the sheet: J1, J2, R?

Commit message: STM32
Parts:
- removed J?: Conn_01x03, symbol Connector_Generic:Conn_01x03
- removed J?: Conn_01x09, symbol Connector_Generic:Conn_01x09
- added C?: 100u, symbol Device:CP_Small
- added C? (x2): 100nF, symbol Device:C_Small
- added D?: RED, symbol Device:LED_Small
- added D? (x6): GREEN, symbol Device:LED_Small
- added D?: ORANGE, symbol Device:LED_Small
- added J?: Conn_01x02, symbol Connector_Generic:Conn_01x02
- added J? (x10): Conn_01x03, symbol Connector_Generic:Conn_01x03
- added J? (x4): Conn_01x05, symbol Connector_Generic:Conn_01x05
- added R?: 47k, symbol Device:R_Small
- added R?: 10k, symbol Device:R_Small
- added R? (x12): 100, symbol Device:R_Small
- added SW?: SW_Push, symbol Switch:SW_Push
- added U? (x3): TSR_1-2425, Converter_DCDC:Converter_DCDC_TRACO_TSR-1_THT, symbol Regulator_Switching:TSR_1-2425
- added U?: TSR_1-2433, Converter_DCDC:Converter_DCDC_TRACO_TSR-1_THT, symbol Regulator_Switching:TSR_1-2433
Connections:
- net GND: now also C?.2, C?.2, C?.2, J?.2 (Pin_2), J?.3 (Pin_3), J?.3 (Pin_3), J?.3 (Pin_3), J?.3 (Pin_3), J?.3 (Pin_3), J?.3 (Pin_3), J?.3 (Pin_3), J?.3 (Pin_3), J?.3 (Pin_3), J?.3 (Pin_3), R?.2, SW?.2, U?.2 (GND), U?.2 (GND), U?.2 (GND), U?.2 (GND)
- net 5V_LIDAR renamed 5V_LIDAR_GP1
- net 5V_LIDAR_GP1: now also U?.3 (Vout); no longer J1.1 (Pin_1), J2.1 (Pin_1), J?.1 (Pin_1), J?.1 (Pin_1)
- new net: J?.1 (Pin_1), R?.2 (x3)
- new net: D?.2 (A), R?.1 (x8)
- new net: C?.1, R?.2, SW?.1
- new net +BATT: C?.1, J?.1 (Pin_1), R?.1, U?.1 (Vin), U?.1 (Vin), U?.1 (Vin), U?.1 (Vin)
- new net 3V3_GPP: R?.1, U?.3 (Vout)
- new net 5V_AUX: J?.2 (Pin_2), J?.2 (Pin_2), J?.2 (Pin_2), R?.2, R?.2, R?.2, R?.2, R?.2, R?.2, R?.2, R?.2, U?.3 (Vout)
- new net 5V_LIDAR_GP2: J1.1 (Pin_1), J2.1 (Pin_1), J?.1 (Pin_1), J?.1 (Pin_1), U?.3 (Vout)
- new net Button1: J?.1 (Pin_1)
- new net Button2: J?.1 (Pin_1)
- new net Button3: J?.1 (Pin_1)
- new net Channel1IN: J?.1 (Pin_1)
- new net Channel1OUT: R?.1
- new net Channel2IN: J?.1 (Pin_1)
- new net Channel2OUT: R?.1
- new net Channel3IN: J?.1 (Pin_1)
- new net Channel3OUT: R?.1
- new net LED1: D?.1 (K)
- new net LED2: D?.1 (K)
- new net LED3: D?.1 (K)
- new net LED4: D?.1 (K)
- new net LED5: D?.1 (K)
- new net LED6: D?.1 (K)
- new net LED7: D?.1 (K)
- new net LED8: D?.1 (K)
- new net RPMSensor: J?.1 (Pin_1)
- new net VBATT_DIV: C?.1, R?.1, R?.2
- new net VBEC: J?.2 (Pin_2), J?.2 (Pin_2), J?.2 (Pin_2), J?.2 (Pin_2), J?.2 (Pin_2), J?.2 (Pin_2), J?.2 (Pin_2)
- no-connect marks 2 -> 0
Other:
- note added: "BT same FTDI RXTX"
- note added: "FTDI"
- note added: "IHM Buttons and LEDS"
- note added: "IMU"
- note added: "IMU and FTDI"
- note added: "LIDAR TF Mini Plus Front Left Right Up"
- note added: "R/C RX and Servo"
- note added: "R/C RX and Servo and Brushless RPM sensor"
- note added: "programming"
- note removed: "LDO 3.3V pour GPS à partir du BEC"
- note removed: "LIDAR"
- note removed: "Partager les liaisons séries de telle sorte que les DMA sont disponible pour le RPLIDAR ou pour les 4 LIDAR"

Commit message: stm32
Parts:
- removed J? (x2): Conn_01x05, symbol Connector_Generic:Conn_01x05
- added C10, C12: 2.2u, symbol Device:C_Small
- added C11, C14, C4, C5, C6, C7, C8, C9: 100nF, symbol Device:C_Small
- added C13: 4.7uF, symbol Device:C_Small
- added H1, H2, H3, H4, H5: MountingHole, symbol Mechanical:MountingHole
- added J16: Conn_01x04, Connectors_JST:JST_SH_SM04B-SRSS-TB_04x1.00mm_Angled, symbol Connector_Generic:Conn_01x04
- added J23: Conn_01x06, symbol Connector_Generic:Conn_01x06
- added J24: Conn_01x07, symbol Connector_Generic:Conn_01x07
- added R23: 10k, symbol Device:R_Small
- added U5: STM32F765VGTx, Package_QFP:LQFP-100_14x14mm_P0.5mm, symbol MCU_ST_STM32F7:STM32F765VGTx
- gave numbers to parts that had none: 57
- renumbered J1 to J13, J2 to J14
Connections:
- net 3V3_GPP: now also J21.1 (Pin_1), C11.1, C13.1, C14.1, C4.1, C5.1, C6.1, C7.1, C8.1, C9.1, U5.100 (VDD), U5.11 (VDD), U5.20 (VREF+), U5.21 (VDDA), U5.27 (VDD), U5.50 (VDD), U5.6 (VBAT), U5.75 (VDD)
- net 5V_AUX: now also J20.4 (Pin_4), J24.2 (Pin_2)
- net Button1: now also U5.15 (PC0)
- net Button2: now also U5.16 (PC1)
- net Button3: now also U5.17 (PC2)
- net Channel1IN: now also U5.39 (PE9)
- net Channel1OUT: now also U5.59 (PD12)
- net Channel2IN: now also U5.30 (PA6)
- net Channel2OUT: now also U5.60 (PD13)
- net Channel3IN: now also U5.22 (PA0)
- net Channel3OUT: now also U5.61 (PD14)
- net GND: now also J20.3 (Pin_3), J21.3 (Pin_3), C10.2, C11.2, C12.2, C13.2, C14.2, C4.2, C5.2, C6.2, C7.2, C8.2, C9.2, J16.4 (Pin_4), J23.1 (Pin_1), J24.1 (Pin_1), J24.6 (Pin_6), R23.2, U5.10 (VSS), U5.19 (VSSA), U5.26 (VSS), U5.49 (VSS), U5.74 (VSS), U5.99 (VSS)
- net LD1_RXi: now also U5.54 (PB15)
- net LD1_TXo: now also U5.53 (PB14)
- net LD2_RXi: now also U5.56 (PD9)
- net LD2_TXo: now also U5.55 (PD8)
- net LD3_RXi: now also U5.64 (PC7)
- net LD3_TXo: now also U5.63 (PC6)
- net LD4_RXi: now also U5.70 (PA11)
- net LD4_TXo: now also U5.71 (PA12)
- net LED1: now also U5.65 (PC8)
- net LED2: now also U5.66 (PC9)
- net LED3: now also U5.78 (PC10)
- net LED4: now also U5.79 (PC11)
- net LED5: now also U5.80 (PC12)
- net LED6: now also U5.7 (PC13)
- net LED7: now also U5.8 (PC14)
- net LED8: now also U5.9 (PC15)
- net RPMSensor: now also U5.4 (PE5)
- net VBEC: now also J16.3 (Pin_3)
- net RESET: now reaches C1.1, R12.2, SW1.1
- net RESET: now also J21.5 (Pin_5), U5.14 (NRST)
- net SWCLK: now reaches J21.2 (Pin_2)
- net SWCLK: now also U5.76 (PA14)
- net SWDIO: now reaches J21.4 (Pin_4)
- net SWDIO: now also U5.72 (PA13)
- net SCL: now reaches J20.1 (Pin_1)
- net SCL: now also U5.92 (PB6)
- net SDA: now reaches J20.2 (Pin_2)
- net SDA: now also U5.93 (PB7)
- new net: C10.1, U5.48 (VCAP_1)
- new net: C12.1, U5.73 (VCAP_2)
- new net: R23.1, U5.94 (BOOT0)
- new net A: J16.1 (Pin_1), U5.23 (PA1)
- new net B: J16.2 (Pin_2), U5.29 (PA5)
- new net BT_RXi: J23.4 (Pin_4), J24.5 (Pin_5), U5.25 (PA3)
- new net BT_TXo: J23.5 (Pin_5), J24.4 (Pin_4), U5.24 (PA2)
- no-connect marks 0 -> 54
Other:
- note added: "Programming"
- note added: "SWD and IMU and FTDI and TELEMETRY"
- note removed: "IMU and FTDI"
- note removed: "programming"
- moved on the sheet: J20, J21

Commit message: stm32
Parts:
- C1, C10, C11, C12, C13, C14, C2, C3, C4, C5, C6, C7, C8, C9: footprint (none) -> Capacitor_SMD:C_0603_1608Metric_Pad1.05x0.95mm_HandSolder
- D1, D2, D3, D4, D5, D6, D7, D8: footprint (none) -> LED_SMD:LED_0805_2012Metric_Pad1.15x1.40mm_HandSolder
- H1, H2, H3, H4, H5: footprint (none) -> MountingHole:MountingHole_3.2mm_M3
- J1, J15, J17, J18, J19, J2, J3, J4, J5, J6: footprint (none) -> Connector_PinHeader_2.54mm:PinHeader_1x03_P2.54mm_Vertical
- J10, J12, J14, J8: footprint Pin_Headers:Pin_Header_Straight_1x04_Pitch2.54mm -> Connector_PinHeader_2.54mm:PinHeader_1x04_P2.54mm_Vertical
- J11, J13, J7, J9: footprint Connectors_JST:JST_SH_SM04B-SRSS-TB_04x1.00mm_Angled -> Connector_JST:JST_SH_BM04B-SRSS-TB_1x04-1MP_P1.00mm_Vertical
- J16: footprint Connectors_JST:JST_SH_SM04B-SRSS-TB_04x1.00mm_Angled -> Connector_PinHeader_2.54mm:PinHeader_1x04_P2.54mm_Vertical
- J20, J21: footprint (none) -> Connector_PinHeader_2.54mm:PinHeader_1x05_P2.54mm_Vertical
- J22: footprint (none) -> Connector_PinHeader_2.54mm:PinHeader_1x02_P2.54mm_Vertical
- J23: footprint (none) -> Connector_PinHeader_2.54mm:PinHeader_1x06_P2.54mm_Vertical
- J24: footprint (none) -> Connector_PinHeader_2.54mm:PinHeader_1x07_P2.54mm_Vertical
- R1, R10, R11, R12, R13, R14, R15, R16, R17, R18, R19, R2, R20, R21, R22, R23, R3, R4, R5, R6, R7, R8, R9: footprint (none) -> Resistor_SMD:R_0603_1608Metric_Pad1.05x0.95mm_HandSolder
- SW1: footprint (none) -> Button_Switch_THT:SW_PUSH_6mm

Commit message: stm32
Parts:
- C2: footprint Capacitor_SMD:C_0603_1608Metric_Pad1.05x0.95mm_HandSolder -> Capacitor_SMD:CP_Elec_8x6.9
Connections:
- net A: now also U5.29 (PA5); no longer U5.23 (PA1)
- net B: now also U5.23 (PA1); no longer U5.29 (PA5)
- net LD3_RXi: now also U5.70 (PA11); no longer U5.64 (PC7)
- net LD3_TXo: now also U5.71 (PA12); no longer U5.63 (PC6)
- net LD4_RXi: now also U5.64 (PC7); no longer U5.70 (PA11)
- net LD4_TXo: now also U5.63 (PC6); no longer U5.71 (PA12)
Changed lines of the file:
@@
 F 0 "C2" H 3488 2296 50  0000 L CNN
 F 1 "100u" H 3488 2205 50  0000 L CNN
-F 2 "Capacitor_SMD:C_0603_1608Metric_Pad1.05x0.95mm_HandSolder" H 3400 2250 50  0001 C CNN
+F 2 "Capacitor_SMD:CP_Elec_8x6.9" H 3400 2250 50  0001 C CNN
 F 3 "~" H 3400 2250 50  0001 C CNN
 	1    3400 2250
@@
 NoConn ~ 10750 3550
 NoConn ~ 10750 3650
+Text Label 12450 6250 0    50   ~ 0
+LD4_RXi
+Text Label 12450 6150 0    50   ~ 0
+LD4_TXo
 Text Label 12450 3250 0    50   ~ 0
-LD4_RXi
+LD3_RXi
 Text Label 12450 3350 0    50   ~ 0
-LD4_TXo
-Text Label 12450 6250 0    50   ~ 0
-LD3_RXi
-Text Label 12450 6150 0    50   ~ 0
 LD3_TXo
 Text Label 10750 6450 2    50   ~ 0
@@
 B
 Text Label 12450 2650 0    50   ~ 0
+A
+Text Label 12450 2250 0    50   ~ 0
 B
-Text Label 12450 2250 0    50   ~ 0
-A
 NoConn ~ 10750 7050
 NoConn ~ 12450 2550

Commit message: stm32
Connections:
- net Channel1IN: now also U5.22 (PA0); no longer U5.39 (PE9)
- net Channel3IN: now also U5.39 (PE9); no longer U5.22 (PA0)
- net LED1: now also U5.9 (PC15); no longer U5.65 (PC8)
- net LED2: now also U5.8 (PC14); no longer U5.66 (PC9)
- net LED3: now also U5.7 (PC13); no longer U5.78 (PC10)
- net LED4: now also U5.5 (PE6); no longer U5.79 (PC11)
- net LED5: now also U5.3 (PE4); no longer U5.80 (PC12)
- net LED6: now also U5.2 (PE3); no longer U5.7 (PC13)
- net LED7: now also U5.1 (PE2); no longer U5.8 (PC14)
- net LED8: now also U5.98 (PE1); no longer U5.9 (PC15)
- net VBATT_DIV: now also U5.31 (PA7)
- no-connect marks 54 -> 53
Other:
- moved on the sheet: C11, C13, C4, C5, C6, C7, C8, C9

Commit message: stm32
Parts:
- R12: value 100 -> 10k
Other:
- moved on the sheet: C10, C12, C14, R23, U5
