File: 20 - STM32_BOARD/stm32_board/GPP.sch (KiCad schematic (older format))
At the start: 80 parts, among them J1 Conn_01x03, J10 Conn_01x04, J11 Conn_01x04, J12 Conn_01x04, J13 Conn_01x04, J14 Conn_01x04, J15 Conn_01x03, J16 Conn_01x04, J17 Conn_01x03, J18 Conn_01x03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

Commit message: stm32
Parts:
- added C15, C16, C17, C19, C20, C21, C22: 100nF, Capacitors_SMD:C_0603_HandSoldering, symbol Device:C_Small
- added C18: 4.7uF, Capacitors_SMD:C_0603_HandSoldering, symbol Device:C_Small
- added J25, J26: Conn_01x01_Female, Pin_Headers:Pin_Header_Straight_1x01_Pitch2.54mm, symbol Connector:Conn_01x01_Female
- C14: footprint Capacitor_SMD:C_0603_1608Metric_Pad1.05x0.95mm_HandSolder -> Capacitors_SMD:C_0603_HandSoldering
Connections:
- net 3V3_GPP: now also C15.1, C16.1, C17.1, C18.1
- net 5V_AUX: now also C19.1, C20.1
- net GND: now also C15.2, C16.2, C17.2, C18.2, C19.2, C20.2, C21.2, C22.2
- net VBEC: now also C21.1, C22.1
- net ADC_spare: now reaches U5.32 (PC4)
- net ADC_spare: now also J25.1 (Pin_1)
- net ChannelspareOUT: now reaches U5.62 (PD15)
- net ChannelspareOUT: now also J26.1 (Pin_1)
- no-connect marks 53 -> 52

Commit message: stm32 & Simu odom
Connections:
- no-connect marks 52 -> 51
Changed lines of the file:
@@
 Text Label 11000 1700 0    50   ~ 0
 B
-NoConn ~ 9300 6500
 NoConn ~ 11000 2000
 NoConn ~ 11000 2400
