File: 20 - STM32_BOARD/stm32_board/stm32_board.kicad_pcb (KiCad board)
At the start: 4 copper layers, 100 x 50 mm, 2 parts, among them J1 Conn_01x04, J2 Conn_01x04

Commit message: stm32
Parts:
- added C1: 100nF, Capacitor_SMD:C_0603_1608Metric_Pad1.05x0.95mm_HandSolder, F.Cu at (119.0, 74.3)
- added C10: 2.2u, Capacitor_SMD:C_0603_1608Metric_Pad1.05x0.95mm_HandSolder, F.Cu at (111.1, 92.0)
- added C11: 100nF, Capacitor_SMD:C_0603_1608Metric_Pad1.05x0.95mm_HandSolder, F.Cu at (106.7, 92.0)
- added C12: 2.2u, Capacitor_SMD:C_0603_1608Metric_Pad1.05x0.95mm_HandSolder, F.Cu at (111.1, 94.6)
- added C13: 4.7uF, Capacitor_SMD:C_0603_1608Metric_Pad1.05x0.95mm_HandSolder, F.Cu at (132.7, 72.1)
- added C14: 100nF, Capacitor_SMD:C_0603_1608Metric_Pad1.05x0.95mm_HandSolder, F.Cu at (119.9, 84.3)
- added C2: 100u, Capacitor_SMD:C_0603_1608Metric_Pad1.05x0.95mm_HandSolder, F.Cu at (69.8, 74.0)
- added C3: 100nF, Capacitor_SMD:C_0603_1608Metric_Pad1.05x0.95mm_HandSolder, F.Cu at (79.3, 71.4)
- added C4: 100nF, Capacitor_SMD:C_0603_1608Metric_Pad1.05x0.95mm_HandSolder, F.Cu at (79.3, 73.9)
- added C5: 100nF, Capacitor_SMD:C_0603_1608Metric_Pad1.05x0.95mm_HandSolder, F.Cu at (129.3, 64.6)
- added C6: 100nF, Capacitor_SMD:C_0603_1608Metric_Pad1.05x0.95mm_HandSolder, F.Cu at (105.6, 87.0)
- added C7: 100nF, Capacitor_SMD:C_0603_1608Metric_Pad1.05x0.95mm_HandSolder, F.Cu at (98.0, 93.0)
- added C8: 100nF, Capacitor_SMD:C_0603_1608Metric_Pad1.05x0.95mm_HandSolder, F.Cu at (98.0, 95.6)
- added C9: 100nF, Capacitor_SMD:C_0603_1608Metric_Pad1.05x0.95mm_HandSolder, F.Cu at (114.4, 81.5)
- added D1: RED, LED_SMD:LED_0805_2012Metric_Pad1.15x1.40mm_HandSolder, F.Cu at (66.0, 105.2)
- added D2: ORANGE, LED_SMD:LED_0805_2012Metric_Pad1.15x1.40mm_HandSolder, F.Cu at (68.6, 105.2)
- added D3: GREEN, LED_SMD:LED_0805_2012Metric_Pad1.15x1.40mm_HandSolder, F.Cu at (71.1, 105.2)
- added D4: GREEN, LED_SMD:LED_0805_2012Metric_Pad1.15x1.40mm_HandSolder, F.Cu at (73.7, 105.2)
- added D5: GREEN, LED_SMD:LED_0805_2012Metric_Pad1.15x1.40mm_HandSolder, F.Cu at (76.2, 105.2)
- added D6: GREEN, LED_SMD:LED_0805_2012Metric_Pad1.15x1.40mm_HandSolder, F.Cu at (78.7, 105.2)
- added D7: GREEN, LED_SMD:LED_0805_2012Metric_Pad1.15x1.40mm_HandSolder, F.Cu at (81.3, 105.2)
- added D8: GREEN, LED_SMD:LED_0805_2012Metric_Pad1.15x1.40mm_HandSolder, F.Cu at (83.8, 105.2)
- added H1: MountingHole, MountingHole:MountingHole_3.2mm_M3, F.Cu at (147.3, 104.1)
- added H2: MountingHole, MountingHole:MountingHole_3.2mm_M3, F.Cu at (53.3, 104.1)
- added H3: MountingHole, MountingHole:MountingHole_3.2mm_M3, F.Cu at (147.3, 147.3)
- added H4: MountingHole, MountingHole:MountingHole_3.2mm_M3, F.Cu at (104.1, 106.7)
- added H5: MountingHole, MountingHole:MountingHole_3.2mm_M3, F.Cu at (53.3, 147.3)
- added J10: Conn_01x04, Connector_PinHeader_2.54mm:PinHeader_1x04_P2.54mm_Vertical, F.Cu at (73.7, 127.0)
- added J11: Conn_01x04, Connector_JST:JST_SH_BM04B-SRSS-TB_1x04-1MP_P1.00mm_Vertical, F.Cu at (63.5, 147.3)
- added J12: Conn_01x04, Connector_PinHeader_2.54mm:PinHeader_1x04_P2.54mm_Vertical, F.Cu at (73.7, 129.5)
- added J13: Conn_01x04, Connector_JST:JST_SH_BM04B-SRSS-TB_1x04-1MP_P1.00mm_Vertical, F.Cu at (73.7, 147.3)
- added J14: Conn_01x04, Connector_PinHeader_2.54mm:PinHeader_1x04_P2.54mm_Vertical, F.Cu at (73.7, 132.1)
- added J15: Conn_01x03, Connector_PinHeader_2.54mm:PinHeader_1x03_P2.54mm_Vertical, F.Cu at (58.4, 134.6)
- added J16: Conn_01x04, Connector_PinHeader_2.54mm:PinHeader_1x04_P2.54mm_Vertical, F.Cu at (61.0, 139.7)
- added J17: Conn_01x03, Connector_PinHeader_2.54mm:PinHeader_1x03_P2.54mm_Vertical, F.Cu at (71.1, 114.3)
- added J18: Conn_01x03, Connector_PinHeader_2.54mm:PinHeader_1x03_P2.54mm_Vertical, F.Cu at (71.1, 116.8)
- added J19: Conn_01x03, Connector_PinHeader_2.54mm:PinHeader_1x03_P2.54mm_Vertical, F.Cu at (71.1, 119.4)
- added J20: Conn_01x05, Connector_PinHeader_2.54mm:PinHeader_1x05_P2.54mm_Vertical, F.Cu at (121.9, 104.1)
- added J21: Conn_01x05, Connector_PinHeader_2.54mm:PinHeader_1x05_P2.54mm_Vertical, F.Cu at (147.3, 127.0)
- added J22: Conn_01x02, Connector_PinHeader_2.54mm:PinHeader_1x02_P2.54mm_Vertical, F.Cu at (137.2, 147.3)
- added J23: Conn_01x06, Connector_PinHeader_2.54mm:PinHeader_1x06_P2.54mm_Vertical, F.Cu at (121.9, 139.7)
- added J24: Conn_01x07, Connector_PinHeader_2.54mm:PinHeader_1x07_P2.54mm_Vertical, F.Cu at (119.4, 139.7)
- added J3: Conn_01x03, Connector_PinHeader_2.54mm:PinHeader_1x03_P2.54mm_Vertical, F.Cu at (58.4, 119.4)
- added J4: Conn_01x03, Connector_PinHeader_2.54mm:PinHeader_1x03_P2.54mm_Vertical, F.Cu at (58.4, 124.5)
- added J5: Conn_01x03, Connector_PinHeader_2.54mm:PinHeader_1x03_P2.54mm_Vertical, F.Cu at (58.4, 127.0)
- added J6: Conn_01x03, Connector_PinHeader_2.54mm:PinHeader_1x03_P2.54mm_Vertical, F.Cu at (58.4, 129.5)
- added J7: Conn_01x04, Connector_JST:JST_SH_BM04B-SRSS-TB_1x04-1MP_P1.00mm_Vertical, F.Cu at (94.0, 147.3)
- added J8: Conn_01x04, Connector_PinHeader_2.54mm:PinHeader_1x04_P2.54mm_Vertical, F.Cu at (73.7, 124.5)
- added J9: Conn_01x04, Connector_JST:JST_SH_BM04B-SRSS-TB_1x04-1MP_P1.00mm_Vertical, F.Cu at (83.8, 147.3)
- added R1: 100, Resistor_SMD:R_0603_1608Metric_Pad1.05x0.95mm_HandSolder, F.Cu at (109.9, 89.5)
- added R10: 100, Resistor_SMD:R_0603_1608Metric_Pad1.05x0.95mm_HandSolder, F.Cu at (128.4, 67.1)
- added R11: 100, Resistor_SMD:R_0603_1608Metric_Pad1.05x0.95mm_HandSolder, F.Cu at (105.6, 89.5)
- added R12: 100, Resistor_SMD:R_0603_1608Metric_Pad1.05x0.95mm_HandSolder, F.Cu at (119.0, 79.3)
- added R13: 47k, Resistor_SMD:R_0603_1608Metric_Pad1.05x0.95mm_HandSolder, F.Cu at (119.0, 76.8)
- added R14: 10k, Resistor_SMD:R_0603_1608Metric_Pad1.05x0.95mm_HandSolder, F.Cu at (114.3, 89.0)
- added R15: 100, Resistor_SMD:R_0603_1608Metric_Pad1.05x0.95mm_HandSolder, F.Cu at (119.9, 81.8)
- added R16: 100, Resistor_SMD:R_0603_1608Metric_Pad1.05x0.95mm_HandSolder, F.Cu at (123.4, 79.3)
- added R17: 100, Resistor_SMD:R_0603_1608Metric_Pad1.05x0.95mm_HandSolder, F.Cu at (114.3, 86.5)
- added R18: 100, Resistor_SMD:R_0603_1608Metric_Pad1.05x0.95mm_HandSolder, F.Cu at (132.7, 69.6)
- added R19: 100, Resistor_SMD:R_0603_1608Metric_Pad1.05x0.95mm_HandSolder, F.Cu at (106.7, 94.6)
- added R2: 100, Resistor_SMD:R_0603_1608Metric_Pad1.05x0.95mm_HandSolder, F.Cu at (115.6, 84.0)
- added R20: 100, Resistor_SMD:R_0603_1608Metric_Pad1.05x0.95mm_HandSolder, F.Cu at (128.4, 72.1)
- added R21: 100, Resistor_SMD:R_0603_1608Metric_Pad1.05x0.95mm_HandSolder, F.Cu at (123.4, 76.8)
- added R22: 100, Resistor_SMD:R_0603_1608Metric_Pad1.05x0.95mm_HandSolder, F.Cu at (102.4, 93.0)
- added R23: 10k, Resistor_SMD:R_0603_1608Metric_Pad1.05x0.95mm_HandSolder, F.Cu at (132.7, 67.1)
- added R3: 100, Resistor_SMD:R_0603_1608Metric_Pad1.05x0.95mm_HandSolder, F.Cu at (127.7, 74.6)
- added R4: 100, Resistor_SMD:R_0603_1608Metric_Pad1.05x0.95mm_HandSolder, F.Cu at (111.2, 84.0)
- added R5: 100, Resistor_SMD:R_0603_1608Metric_Pad1.05x0.95mm_HandSolder, F.Cu at (109.9, 87.0)
- added R6: 100, Resistor_SMD:R_0603_1608Metric_Pad1.05x0.95mm_HandSolder, F.Cu at (123.4, 74.3)
- added R7: 100, Resistor_SMD:R_0603_1608Metric_Pad1.05x0.95mm_HandSolder, F.Cu at (102.4, 95.6)
- added R8: 100, Resistor_SMD:R_0603_1608Metric_Pad1.05x0.95mm_HandSolder, F.Cu at (128.4, 69.6)
- added R9: 100, Resistor_SMD:R_0603_1608Metric_Pad1.05x0.95mm_HandSolder, F.Cu at (133.7, 64.6)
- added SW1: SW_Push, Button_Switch_THT:SW_PUSH_6mm, F.Cu at (147.3, 111.8)
- added U1: TSR_1-2425, Converter_DCDC:Converter_DCDC_TRACO_TSR-1_THT, F.Cu at (134.6, 137.2)
- added U2: TSR_1-2425, Converter_DCDC:Converter_DCDC_TRACO_TSR-1_THT, F.Cu at (134.6, 116.8)
- added U3: TSR_1-2433, Converter_DCDC:Converter_DCDC_TRACO_TSR-1_THT, F.Cu at (134.6, 106.7)
- added U4: TSR_1-2425, Converter_DCDC:Converter_DCDC_TRACO_TSR-1_THT, F.Cu at (134.6, 127.0)
- added U5: STM32F765VGTx, Package_QFP:LQFP-100_14x14mm_P0.5mm, F.Cu at (99.1, 129.5)
- J1: value Conn_01x04 -> Conn_01x03; footprint Connectors_JST:JST_SH_SM04B-SRSS-TB_04x1.00mm_Angled -> Connector_PinHeader_2.54mm:PinHeader_1x03_P2.54mm_Vertical
- J2: value Conn_01x04 -> Conn_01x03; footprint Pin_Headers:Pin_Header_Straight_1x04_Pitch2.54mm -> Connector_PinHeader_2.54mm:PinHeader_1x03_P2.54mm_Vertical
- moved J2 8.98 mm to (58.4, 116.8), turned to 270 degrees
- moved J1 6.17 mm to (58.4, 114.3)
Connections:
- net /GPP/LD1_RXi renamed /GPP/VBEC
- J1 pad 1: /GPP/5V_LIDAR -> /GPP/Channel1IN
- J1 pad 3: /GPP/LD1_TXo -> GND
- J2 pad 1: /GPP/5V_LIDAR -> /GPP/Channel2IN
- J2 pad 3: /GPP/LD1_TXo -> GND

Commit message: stm32
Parts:
- C2: footprint Capacitor_SMD:C_0603_1608Metric_Pad1.05x0.95mm_HandSolder -> Capacitor_SMD:CP_Elec_8x6.9
- moved C2 97.2 mm to (144.8, 135.9), turned to 270 degrees
- moved C4 89.3 mm to (161.3, 109.2)
- moved R3 85.8 mm to (61.8, 129.5), turned to 180 degrees
- moved C3 84.0 mm to (146.4, 121.9)
- moved R9 81.8 mm to (100.3, 139.3), turned to 270 degrees
- moved R10 81.5 mm to (91.4, 139.7), turned to 270 degrees
- moved R6 79.2 mm to (78.7, 139.7), turned to 270 degrees
- moved C5 78.1 mm to (163.8, 134.6)
- moved R8 73.8 mm to (104.1, 139.3), turned to 270 degrees
- moved R18 72.6 mm to (68.6, 103.7), turned to 90 degrees
- moved R4 70.9 mm to (67.3, 139.7), turned to 270 degrees
- moved R5 69.4 mm to (64.8, 139.7), turned to 270 degrees
- moved R2 68.8 mm to (61.8, 127.0), turned to 180 degrees
- moved C6 67.6 mm to (163.4, 121.9)
- moved C7 66.7 mm to (161.7, 113.0)
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Connections:
- U5 pad 23: /GPP/A -> /GPP/B
- U5 pad 29: /GPP/B -> /GPP/A
- U5 pad 63: /GPP/LD3_TXo -> /GPP/LD4_TXo
- U5 pad 64: /GPP/LD3_RXi -> /GPP/LD4_RXi
- U5 pad 70: /GPP/LD4_RXi -> /GPP/LD3_RXi
- U5 pad 71: /GPP/LD4_TXo -> /GPP/LD3_TXo
Routing:
- net GND: track 0.00 -> 260.1 mm, vias 0 -> 9
- net /GPP/5V_AUX: track 0.00 -> 138.6 mm
- net /GPP/5V_LIDAR_GP1: track 0.00 -> 83.7 mm, vias 0 -> 2
- net +BATT: track 0.00 -> 65.2 mm
- net /GPP/5V_LIDAR_GP2: track 0.00 -> 50.1 mm, vias 0 -> 2
- net /GPP/RPMSensor: track 0.00 -> 49.4 mm, vias 0 -> 1
- net /GPP/BT_RXi: track 0.00 -> 48.5 mm, vias 0 -> 1
- net /GPP/BT_TXo: track 0.00 -> 46.0 mm, vias 0 -> 1
- net /GPP/B: track 0.00 -> 41.6 mm
- net /GPP/SCL: track 0.00 -> 37.1 mm
- net /GPP/Channel3OUT: track 0.00 -> 33.3 mm, vias 0 -> 2
- net /GPP/SDA: track 0.00 -> 31.7 mm
- net /GPP/Channel2OUT: track 0.00 -> 31.0 mm, vias 0 -> 2
- net /GPP/A: track 0.00 -> 30.9 mm
- net /GPP/Channel1OUT: track 0.00 -> 28.8 mm, vias 0 -> 2
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- added copper zone on In2.Cu, net /GPP/3V3_GPP
- added copper zone on In1.Cu, net GND

Commit message: stm32
Parts:
- C11, C4, C5, C7: moved to B.Cu
- moved C6 87.8 mm to (76.2, 131.7), turned to 90 degrees
- moved C8 85.5 mm to (77.5, 119.0), turned to 90 degrees
- moved C11 75.2 mm to (87.4, 119.4)
- moved C7 74.7 mm to (87.4, 120.7)
- moved C5 74.3 mm to (90.8, 120.7), turned to 180 degrees
- moved C4 71.2 mm to (90.8, 119.4)
- moved C9 65.1 mm to (97.8, 133.7), turned to 270 degrees
- moved C13 62.8 mm to (100.6, 116.2)
- moved C14 3.82 mm to (100.6, 118.1)
- moved C12 1.91 mm to (98.0, 136.5)
- moved R23 1.28 mm to (100.6, 120.7), turned to 0 degrees
- moved C10 0.90 mm to (77.1, 128.9)
Connections:
- U5 pad 1: Net-(U5-Pad1) -> /GPP/LED7
- U5 pad 2: Net-(U5-Pad2) -> /GPP/LED6
- U5 pad 22: /GPP/Channel3IN -> /GPP/Channel1IN
- U5 pad 3: Net-(U5-Pad3) -> /GPP/LED5
- U5 pad 31: Net-(U5-Pad31) -> /GPP/VBATT_DIV
- U5 pad 39: /GPP/Channel1IN -> /GPP/Channel3IN
- U5 pad 5: Net-(U5-Pad5) -> /GPP/LED4
- U5 pad 65: /GPP/LED1 -> Net-(U5-Pad65)
- U5 pad 66: /GPP/LED2 -> Net-(U5-Pad66)
- U5 pad 7: /GPP/LED6 -> /GPP/LED3
- U5 pad 78: /GPP/LED3 -> Net-(U5-Pad78)
- U5 pad 79: /GPP/LED4 -> Net-(U5-Pad79)
- U5 pad 8: /GPP/LED7 -> /GPP/LED2
- U5 pad 80: /GPP/LED5 -> Net-(U5-Pad80)
- U5 pad 9: /GPP/LED8 -> /GPP/LED1
- U5 pad 98: Net-(U5-Pad98) -> /GPP/LED8
Routing:
- net /GPP/RESET: track 17.7 -> 93.0 mm, vias 0 -> 1
- net /GPP/VBATT_DIV: track 4.60 -> 68.3 mm, vias 0 -> 2
- net /GPP/3V3_GPP: track 2.06 -> 43.3 mm, vias 1 -> 9
- net /GPP/LED1: track 0.00 -> 35.0 mm
- net /GPP/Channel1IN: track 0.00 -> 35.0 mm
- net /GPP/LED2: track 0.00 -> 33.1 mm
- net /GPP/LED3: track 0.00 -> 31.1 mm
- net /GPP/SWDIO: track 0.00 -> 30.8 mm, vias 0 -> 1
- net /GPP/LED4: track 0.00 -> 29.7 mm
- net GND: track 260.1 -> 289.5 mm, vias 9 -> 17
- net /GPP/LED5: track 0.00 -> 28.0 mm
- net /GPP/SWCLK: track 0.00 -> 27.8 mm, vias 0 -> 1
- net /GPP/LED8: track 0.00 -> 26.2 mm
- net /GPP/LED6: track 0.00 -> 26.0 mm
- net /GPP/Channel2IN: track 0.00 -> 25.5 mm, vias 0 -> 1
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Other:
- board text added: "+"
- board text added: "-"
- board text added: "1"
- board text added: "A/B"
- board text added: "BUTTON123"
- board text added: "Bluetooth"
- board text added: "DEBUG"
- board text added: "FTDI Cable"
- board text added: "IMU MinIMU9-v5"
- board text added: "RCIN123"
- board text added: "RPM"
- board text added: "SERVO123"
- board text added: "s"

Commit message: stm32
Parts:
- moved C6 1.27 mm to (77.5, 131.7)
- moved H4 0.96 mm to (102.0, 105.0)
Routing:
- net /GPP/VBATT_DIV: track 68.3 -> 93.9 mm
- net /GPP/VBEC: track 25.4 -> 50.8 mm
- net GND: track 289.5 -> 314.3 mm
Other:
- board text added: "< LIDAR TF mini Plus 1234"
- board text added: "Bluetooth Module"
- board text added: "RESET"
- board text added: "STM32 Controller TRR 2020 Roulant"
- board text removed: "Bluetooth"
