File: 20 - STM32_BOARD/stm32_board/stm32_board.kicad_pcb (KiCad board)
At the start: 4 copper layers, 100 x 50 mm, 80 parts, among them J1 Conn_01x03, J10 Conn_01x04, J11 Conn_01x04, J12 Conn_01x04, J13 Conn_01x04, J14 Conn_01x04, J15 Conn_01x03, J16 Conn_01x04, J17 Conn_01x03, J18 Conn_01x03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

Commit message: stm32
Parts:
- added C15: 100nF, Capacitors_SMD:C_0603_HandSoldering, F.Cu at (100.6, 130.0)
- added C16: 100nF, Capacitors_SMD:C_0603_HandSoldering, F.Cu at (93.5, 108.2)
- added C17: 100nF, Capacitors_SMD:C_0603_HandSoldering, B.Cu at (129.5, 121.9)
- added C18: 4.7uF, Capacitors_SMD:C_0603_HandSoldering, F.Cu at (75.7, 131.8)
- added C19: 100nF, Capacitors_SMD:C_0603_HandSoldering, F.Cu at (118.9, 110.7)
- added C20: 100nF, Capacitors_SMD:C_0603_HandSoldering, F.Cu at (120.9, 138.7)
- added C21: 100nF, Capacitors_SMD:C_0603_HandSoldering, F.Cu at (54.4, 121.9)
- added C22: 100nF, Capacitors_SMD:C_0603_HandSoldering, F.Cu at (54.4, 132.1)
- added J25: Conn_01x01_Female, Pin_Headers:Pin_Header_Straight_1x01_Pitch2.54mm, F.Cu at (75.7, 126.0)
- added J26: Conn_01x01_Female, Pin_Headers:Pin_Header_Straight_1x01_Pitch2.54mm, F.Cu at (72.1, 128.5)
- C14: footprint Capacitor_SMD:C_0603_1608Metric_Pad1.05x0.95mm_HandSolder -> Capacitors_SMD:C_0603_HandSoldering
- R12: value 100 -> 10k
- moved H3 0.97 mm to (146.0, 146.0)
- moved H5 0.95 mm to (54.0, 146.0)
- moved H1 0.85 mm to (146.0, 104.0)
- moved H2 0.82 mm to (54.0, 104.0)
Connections:
- J20 pad 5: Net-(J20-Pad5) -> (no net)
- J23 pad 2: Net-(J23-Pad2) -> (no net)
- J23 pad 3: Net-(J23-Pad3) -> (no net)
- J23 pad 6: Net-(J23-Pad6) -> (no net)
- J24 pad 3: Net-(J24-Pad3) -> (no net)
- J24 pad 7: Net-(J24-Pad7) -> (no net)
- U5 pad 12: Net-(U5-Pad12) -> (no net)
- U5 pad 13: Net-(U5-Pad13) -> (no net)
- U5 pad 18: Net-(U5-Pad18) -> (no net)
- U5 pad 28: Net-(U5-Pad28) -> (no net)
- U5 pad 32: Net-(U5-Pad32) -> /GPP/ADC_spare
- U5 pad 33: Net-(U5-Pad33) -> (no net)
- U5 pad 34: Net-(U5-Pad34) -> (no net)
- U5 pad 35: Net-(U5-Pad35) -> (no net)
- U5 pad 36: Net-(U5-Pad36) -> (no net)
- U5 pad 37: Net-(U5-Pad37) -> (no net)
- U5 pad 38: Net-(U5-Pad38) -> (no net)
- U5 pad 40: Net-(U5-Pad40) -> (no net)
- U5 pad 41: Net-(U5-Pad41) -> (no net)
- U5 pad 42: Net-(U5-Pad42) -> (no net)
- U5 pad 43: Net-(U5-Pad43) -> (no net)
- U5 pad 44: Net-(U5-Pad44) -> (no net)
- U5 pad 45: Net-(U5-Pad45) -> (no net)
- U5 pad 46: Net-(U5-Pad46) -> (no net)
- U5 pad 47: Net-(U5-Pad47) -> (no net)
- U5 pad 51: Net-(U5-Pad51) -> (no net)
- U5 pad 52: Net-(U5-Pad52) -> (no net)
- U5 pad 57: Net-(U5-Pad57) -> (no net)
- U5 pad 58: Net-(U5-Pad58) -> (no net)
- U5 pad 62: Net-(U5-Pad62) -> /GPP/ChannelspareOUT
- U5 pad 65: Net-(U5-Pad65) -> (no net)
- U5 pad 66: Net-(U5-Pad66) -> (no net)
- U5 pad 67: Net-(U5-Pad67) -> (no net)
- U5 pad 68: Net-(U5-Pad68) -> (no net)
- U5 pad 69: Net-(U5-Pad69) -> (no net)
- U5 pad 77: Net-(U5-Pad77) -> (no net)
- U5 pad 78: Net-(U5-Pad78) -> (no net)
- U5 pad 79: Net-(U5-Pad79) -> (no net)
- U5 pad 80: Net-(U5-Pad80) -> (no net)
- U5 pad 81: Net-(U5-Pad81) -> (no net)
- U5 pad 82: Net-(U5-Pad82) -> (no net)
- U5 pad 83: Net-(U5-Pad83) -> (no net)
- U5 pad 84: Net-(U5-Pad84) -> (no net)
- U5 pad 85: Net-(U5-Pad85) -> (no net)
- U5 pad 86: Net-(U5-Pad86) -> (no net)
- U5 pad 87: Net-(U5-Pad87) -> (no net)
- U5 pad 88: Net-(U5-Pad88) -> (no net)
- U5 pad 89: Net-(U5-Pad89) -> (no net)
- U5 pad 90: Net-(U5-Pad90) -> (no net)
- U5 pad 91: Net-(U5-Pad91) -> (no net)
- U5 pad 95: Net-(U5-Pad95) -> (no net)
- U5 pad 96: Net-(U5-Pad96) -> (no net)
- U5 pad 97: Net-(U5-Pad97) -> (no net)
Routing:
- net GND: track 314.3 -> 362.3 mm, vias 17 -> 19
- net /GPP/ChannelspareOUT: track 0.00 -> 19.8 mm, vias 0 -> 1
- net /GPP/5V_AUX: track 137.2 -> 147.6 mm
- net /GPP/3V3_GPP: track 43.2 -> 51.4 mm, vias 9 -> 10
- net /GPP/ADC_spare: track 0.00 -> 7.41 mm
- net /GPP/B: track 42.9 -> 40.0 mm
- net /GPP/RPMSensor: track 53.0 -> 54.4 mm
- net /GPP/A: track 31.4 -> 30.2 mm

Commit message: stm32 & Simu odom
Parts:
- moved J26 0.51 mm to (71.6, 128.5)
- moved R1 0.28 mm to (62.1, 124.5)
- moved R2 0.28 mm to (62.1, 127.0)
- moved R3 0.28 mm to (62.1, 129.5)
- moved C5 0.25 mm to (90.8, 120.9)
- moved C7 0.25 mm to (87.4, 120.9)
Routing:
- net GND: track 362.3 -> 448.2 mm, vias 19 -> 20
- net +BATT: track 65.2 -> 140.3 mm, vias 0 -> 1
- net /GPP/ChannelspareOUT: track 19.8 -> 19.0 mm
